Commit message: modify kinect cam

File: src/my_robot/urdf/cam_robot.xacro (robot description, xacro)
@@ -121,5 +121,5 @@
     <dynamics damping="1.0" friction="1.0"/>
   </joint>
-  <link name="camera">
+  <link name="camera_link">
     <inertial>
       <mass value="0.1"/>
@@ -131,5 +131,5 @@
       />
     </inertial>
-    <collision name='camera_collision'>
+    <collision name='camera_link_collision'>
       <origin xyz="0 0 0" rpy="0 0 0"/>
       <geometry>
@@ -138,5 +138,5 @@
       <box_inertia m="0.1" x="0.05" y="0.05" z="0.05"/>
     </collision>
-    <visual name='camera_visual'>
+    <visual name='camera_link_visual'>
       <origin xyz="0 0 0" rpy="0 0 0"/>
       <geometry>
@@ -146,8 +146,8 @@
     </visual>
   </link>
-  <joint type="fixed" name="camera_joint">
+  <joint type="fixed" name="camera_link_joint">
     <origin xyz="0.3 0 0" rpy="0 0 0"/>
-    <child link="camera"/>
-    <parent link="chassis"/>
+    <child link="camera_link"/>
+    <parent link="camera_link_optical"/>
     <axis xyz="0 1 0"/>
   </joint>
@@ -181,3 +181,31 @@
     <axis xyz="0 1 0" rpy="0 0 0"/>
   </joint>
+  <link name="camera_link_optical">
+  <inertial>
+      <mass value="0.1"/>
+      <origin xyz="0 0.4 0" rpy="0 0 0"/>
+      <inertia
+        ixx="1e-6" ixy="0" ixz="0"
+        iyy="1e-6" iyz="0"
+        izz="1e-6"
+      />
+  </inertial>
+    <collision name='camera_link_optical_collision'>
+      <origin xyz="0 0.4 0" rpy="0 0 0"/>
+      <geometry>
+        <box size="0.3 0.05 0.05"/>
+      </geometry>
+    </collision>
+    <visual name='camera_link_optical_visual'>
+      <origin xyz="0 0.4 0" rpy="0 0 0"/>
+      <geometry>
+        <mesh filename="package://my_robot/meshes/kinect.dae"/>
+      </geometry>
+    </visual>
+  </link>
+  <joint name="camera_optical_joint" type="fixed">
+    <origin xyz="0 0 0" rpy="-1.5707 0 -1.5707"/>
+    <parent link="chassis"/>
+    <child link="camera_link_optical"/>
+  </joint>
 </robot>

Commit message: change camera_optical_link

File: src/my_robot/urdf/cam_robot.xacro (robot description, xacro)
@@ -105,4 +105,29 @@
     </collision>
   </link>
+  <link name="camera_link">
+    <inertial>
+      <mass value="0.1"/>
+      <origin xyz="0 0 0" rpy="0 0 0"/>
+      <inertia
+        ixx="1e-6" ixy="0" ixz="0"
+        iyy="1e-6" iyz="0"
+        izz="1e-6"
+      />
+    </inertial>
+    <collision name='camera_link_collision'>
+      <origin xyz="0 0 0" rpy="0 0 0"/>
+      <geometry>
+        <box size="0.05 0.05 0.05"/>
+      </geometry>
+      <box_inertia m="0.1" x="0.05" y="0.05" z="0.05"/>
+    </collision>
+    <visual name='camera_link_visual'>
+      <origin xyz="0 0 0" rpy="0 0 0"/>
+      <geometry>
+        <box size="0.1 0.1 0.1"/>
+      </geometry>
+      <box_inertia m="0.1" x="0.05" y="0.05" z="0.05"/>
+    </visual>
+  </link>
   <joint type="continuous" name="left_wheel_hinge">
     <origin xyz="0 0.2 0"/>
@@ -121,8 +146,14 @@
     <dynamics damping="1.0" friction="1.0"/>
   </joint>
-  <link name="camera_link">
-    <inertial>
-      <mass value="0.1"/>
-      <origin xyz="0.3 0 0" rpy="0 0 0"/>
+  <joint type="fixed" name="camera_link_joint">
+    <origin xyz="0.2 0 0" rpy="0 0 0"/>
+    <child link="camera_link"/>
+    <parent link="chassis"/>
+    <axis xyz="0 1 0"/>
+  </joint>
+  <link name="hokuyo">
+    <inertial>
+      <mass value="1e-5"/>
+      <origin xyz="0 0 0" rpy="0 0 0"/>
       <inertia
         ixx="1e-6" ixy="0" ixz="0"
@@ -131,28 +162,26 @@
       />
     </inertial>
-    <collision name='camera_link_collision'>
-      <origin xyz="0 0 0" rpy="0 0 0"/>
-      <geometry>
-        <box size="0.05 0.05 0.05"/>
-      </geometry>
-      <box_inertia m="0.1" x="0.05" y="0.05" z="0.05"/>
-    </collision>
-    <visual name='camera_link_visual'>
+    <collision name='hokuyo_collision'>
       <origin xyz="0 0 0" rpy="0 0 0"/>
       <geometry>
         <box size="0.1 0.1 0.1"/>
       </geometry>
-      <box_inertia m="0.1" x="0.05" y="0.05" z="0.05"/>
-    </visual>
-  </link>
-  <joint type="fixed" name="camera_link_joint">
-    <origin xyz="0.3 0 0" rpy="0 0 0"/>
-    <child link="camera_link"/>
-    <parent link="camera_link_optical"/>
-    <axis xyz="0 1 0"/>
-  </joint>
-  <link name="hokuyo">
-    <inertial>
-      <mass value="1e-5"/>
+    </collision>
+    <visual name='hokuyo_visual'>
+      <origin xyz="0 0 0" rpy="0 0 0"/>
+      <geometry>
+        <mesh filename="package://my_robot/meshes/hokuyo.dae"/>
+      </geometry>
+    </visual>
+  </link>
+  <joint type="fixed" name="hokuyo_joint">
+    <origin xyz="0.15 0 0.2" rpy="0 0 0"/>
+    <child link="hokuyo"/>
+    <parent link="chassis"/>
+    <axis xyz="0 1 0" rpy="0 0 0"/>
+  </joint>
+  <link name="camera_link_optical">
+  <inertial>
+      <mass value="0.2"/>
       <origin xyz="0 0 0" rpy="0 0 0"/>
       <inertia
@@ -161,51 +190,25 @@
         izz="1e-6"
       />
-    </inertial>
-    <collision name='hokuyo_collision'>
-      <origin xyz="0 0 0" rpy="0 0 0"/>
-      <geometry>
-        <box size="0.1 0.1 0.1"/>
-      </geometry>
-    </collision>
-    <visual name='hokuyo_visual'>
-      <origin xyz="0 0 0" rpy="0 0 0"/>
-      <geometry>
-        <mesh filename="package://my_robot/meshes/hokuyo.dae"/>
-      </geometry>
-    </visual>
-  </link>
-  <joint type="fixed" name="hokuyo_joint">
-    <origin xyz="0.2 0 0.1" rpy="0 0 0"/>
-    <child link="hokuyo"/>
-    <parent link="chassis"/>
-    <axis xyz="0 1 0" rpy="0 0 0"/>
-  </joint>
-  <link name="camera_link_optical">
-  <inertial>
-      <mass value="0.1"/>
-      <origin xyz="0 0.4 0" rpy="0 0 0"/>
-      <inertia
-        ixx="1e-6" ixy="0" ixz="0"
-        iyy="1e-6" iyz="0"
-        izz="1e-6"
-      />
   </inertial>
     <collision name='camera_link_optical_collision'>
-      <origin xyz="0 0.4 0" rpy="0 0 0"/>
-      <geometry>
-        <box size="0.3 0.05 0.05"/>
-      </geometry>
+      <origin xyz="0 0 0" rpy="0 0 0"/>
+      <geometry>
+        <box size="0 0.2 0.05"/>
+      </geometry>
+      <box_inertia m="0.2" x="0.05" y="0.05" z="0.05"/>
     </collision>
     <visual name='camera_link_optical_visual'>
-      <origin xyz="0 0.4 0" rpy="0 0 0"/>
+      <origin xyz="0 0 0" rpy="0 0 0"/>
       <geometry>
         <mesh filename="package://my_robot/meshes/kinect.dae"/>
       </geometry>
+      <box_inertia m="0.2" x="0.05" y="0.05" z="0.05"/>
     </visual>
   </link>
   <joint name="camera_optical_joint" type="fixed">
-    <origin xyz="0 0 0" rpy="-1.5707 0 -1.5707"/>
+    <origin xyz="0 0 0.2" rpy="0 0 0"/>
     <parent link="chassis"/>
     <child link="camera_link_optical"/>
+    <axis xyz="0 0 1" rpy="0 0 0"/>
   </joint>
 </robot>
